File: ArduinoDemoBoard.kicad_sch (KiCad schematic)
At the start: 5 parts, among them M1 Motor_Servo, U1 HC-SR04, U2 NHD-C0220BIZ

Commit message: Kommentar
Parts:
- U2: value NHD-C0220BIZ -> 2x16 lcd display
Changed lines of the file:
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@@
 			)
 		)
-		(property "Value" "NHD-C0220BIZ"
+		(property "Value" "2x16 lcd display"
 			(at 75.4065 20.32 0)
 			(effects
